Commit message: Fixed scaling on URDF

File: robots/youbot_arm.urdf.xacro (robot description, xacro)
@@ -32,4 +32,7 @@
     </inertial>
     </link>
+    <gazebo reference="base_link">
+		   <material>youbot/Orange</material>
+    </gazebo>
   <xacro:youbot_arm name="arm" parent="base_link">
     <origin xyz="0 0 0" rpy="0 0 0" />

File: robots/youbot_gripper.urdf.xacro (robot description, xacro)
@@ -25,4 +25,7 @@
   <link name="base_link">
   </link>
+  <gazebo reference="base_link">
+       <material>youbot/DarkGrey</material>
+  </gazebo>
   <xacro:youbot_gripper name="gripper" parent="base_link">
     <origin xyz="0 0 0" rpy="0 0 0" />

File: urdf/youbot_arm/arm.urdf.xacro (robot description, xacro)
@@ -37,4 +37,7 @@
 			</collision>
 		</link>
+		<gazebo reference = "${name}_link_0">
+			<material>DarkGrey</material>
+		</gazebo>
 		<!-- joint between arm_0_link and arm_1_link -->
 		<joint name="${name}_joint_1" type="revolute">
@@ -76,4 +79,7 @@
 			</collision>
 		</link>
+		<gazebo reference = "${name}_link_1">
+			<material>Orange</material>
+		</gazebo>
 		<!-- joint between arm_1_link and arm_2_link -->
 		<joint name="${name}_joint_2" type="revolute">
@@ -108,4 +114,7 @@
 			</collision>
 		</link>
+		<gazebo reference = "${name}_link_2">
+			<material>Orange</material>
+		</gazebo>
 		<!-- joint between arm_2_link and arm_3_link -->
 		<!--<joint name="${name}_joint_3" type="revolute">
@@ -148,4 +157,7 @@
 			</collision>
 		</link>
+		<gazebo reference = "${name}_link_3">
+			<material>Orange</material>
+		</gazebo>
 		<!-- joint between arm_3_link and arm_4_link -->
 		<joint name="${name}_joint_4" type="revolute">
@@ -180,4 +192,7 @@
 			</collision>
 		</link>
+		<gazebo reference = "${name}_link_4">
+			<material>Orange</material>
+		</gazebo>
 		<!-- joint between arm_4_link and arm_5_link -->
 		<joint name="${name}_joint_5" type="revolute">
@@ -211,4 +226,7 @@
 			</collision>
 		</link>
+		<gazebo reference = "${name}_link_5">
+			<material>DarkGrey</material>
+		</gazebo>
 		<!-- extensions -->
 		<xacro:youbot_arm_gazebo name="${name}" />

File: urdf/youbot_base/base.urdf.xacro (robot description, xacro)
@@ -252,4 +252,7 @@
       				</inertial>
    		</link>
+		<gazebo reference = "caster_link_br">
+			<material>Orange</material>
+		</gazebo>
 		<joint name="wheel_joint_br" type="continuous">
       			<axis xyz="0 1 0" />
@@ -283,4 +286,7 @@
       			</collision>
     		</link>
+		<gazebo reference = "wheel_link_br">
+			<material>Orange</material>
+		</gazebo>
 	<!-- extensions -->
 		<xacro:youbot_base_gazebo />

File: urdf/youbot_gripper/gripper.urdf.xacro (robot description, xacro)
@@ -35,4 +35,7 @@
 			</collision>
 		</link>
+		<gazebo reference = "${name}_palm_link">
+			<material>Black</material>
+		</gazebo>
 		<joint name="${name}_finger_joint_l" type="prismatic">
 			<origin xyz="0.004 0.008 0.046" rpy="0 0 ${M_PI}" />
@@ -65,4 +68,7 @@
 			</collision>
 		</link>
+		<gazebo reference = "${name}_finger_link_l">
+			<material>Black</material>
+		</gazebo>
                <joint name="${name}_finger_joint_r" type="prismatic">
 			<origin xyz="0.004 -0.008 0.046" rpy="0 0 0" />
@@ -95,4 +101,7 @@
 			</collision>
 		</link>
+		<gazebo reference = "${name}_finger_link_r">
+			<material>Black</material>
+		</gazebo>
 		<!-- extensions -->
 		<xacro:youbot_gripper_gazebo name="${name}" />

File: urdf/youbot_plate/plate.urdf.xacro (robot description, xacro)
@@ -31,4 +31,7 @@
 			</collision>
 		</link>
+		<gazebo reference = "${name}_link">
+			<material>DarkGrey</material>
+		</gazebo>
 		<!-- extensions -->
 	</xacro:macro>
