Commit message: added asus camera to gripper urdf

File: robots/youbot-sensors.urdf.xacro (robot description, xacro)
@@ -55,9 +55,7 @@
   </xacro:sensor_angle>
   <!-- ASUS Xtion on arm sensor angle -->
-<!--
-  <xacro:asus_xtion_camera name="openni" parent="arm_sensor_angle_part2_link"  tilt="0.0">
+  <!-- <xacro:asus_xtion_camera name="openni" parent="arm_sensor_angle_part2_link"  tilt="0.0">
     <origin xyz="0.01 0.0 0.0" rpy="${M_PI} 0.0 ${M_PI}" />
-  </xacro:asus_xtion_camera>
--->
+  </xacro:asus_xtion_camera> -->
   <!-- tower -->
 <!--

File: urdf/sensors/asus_xtion_camera.urdf.xacro (robot description, xacro)
@@ -68,7 +68,7 @@
      	<parent link="${name}_foot_link"/>
      	<child link="${name}_tilt_link"/>
-     	<!--<axis xyz="0 1 0"/>-->
-      	<origin xyz="0 0 0.0075" rpy="0 ${tilt} 0"/>
-		<!--<limit effort="100" lower="-0.541052068" upper="0.541052068" velocity="1.0"/>-->
+   	<!--<axis xyz="0 1 0"/>-->
+    	<origin xyz="0 0 0.0075" rpy="0 ${tilt} 0"/>
+	<!--<limit effort="100" lower="-0.541052068" upper="0.541052068" velocity="1.0"/>-->
     </joint>
     <link name="${name}_camera">

File: urdf/youbot_base/base.urdf.xacro (robot description, xacro)
@@ -84,5 +84,5 @@
 		<!-- base laser front -->
     		<xacro:hokuyo_urg04_laser name="${name}_laser_front" parent="${name}" ros_topic="scan_front" update_rate="10" min_angle="-1.57" max_angle="1.57" >
-     			 <origin xyz="0.3 0 -0.03" rpy="0 0 0" />
+     			 <origin xyz="0.3 0 -0.03" rpy="3.14 0 0" />
     		</xacro:hokuyo_urg04_laser>
 	<!-- front left wheel -->

File: urdf/youbot_gripper/gripper.urdf.xacro (robot description, xacro)
@@ -7,4 +7,5 @@
 	<include filename="$(find youbot_description)/urdf/youbot_gripper/gripper.transmission.xacro" />
 	<include filename="$(find youbot_description)/urdf/youbot_gripper/limits.urdf.xacro" />
+	<include filename="$(find youbot_description)/urdf/sensors/asus_xtion_camera.urdf.xacro" />
 	<xacro:macro name="youbot_gripper" params="parent name *origin">
 		<!-- joint between arm_7_link and sdh_palm_link -->
@@ -95,4 +96,8 @@
 			</collision>
 		</link>
+		<!-- asus xtion camera -->
+		<xacro:asus_xtion_camera name="openni" parent="gripper_palm_link" tilt="0.0">
+		  <origin xyc="0.01 0.0 0.0" rpy="0 ${M_PI/2} 0.0" />
+                </xacro:asus_xtion_camera>
 		<!-- extensions -->
 		<xacro:youbot_gripper_gazebo name="${name}" />
