Commit message: Transitioning to more current URDF of youbot from youbot-store, Still WIP

File: robots/youbot.urdf (robot description, URDF)
Before this commit: robot youbot, 11 links, 10 joints
Links:
- added link ar_marker_fixed; visual box size=0.11 0.11 0.003
- added link base_footprint, mass 0.0001; collision box size=0.001 0.001 0.001; visual box size=0.001 0.001 0.001
- added link base_laser_front_link, mass 0.16; collision mesh filename=package://youbot_description/meshes/sensors/hokuyo_convex.d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; visual mesh filename=package://youbot_description/meshes/sensors/hokuyo.dae
- added link caster_link_bl, mass 0.1
- added link caster_link_br, mass 0.1
- added link caster_link_fl, mass 0.1
- added link caster_link_fr, mass 0.1
- added link plate_link, mass 1; collision mesh filename=package://youbot_description/meshes/youbot_plate/plate_conv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; visual mesh filename=package://youbot_description/meshes/youbot_plate/plate.dae
- added link wheel_link_bl, mass 0.4; collision cylinder length=0.05 radius=0.05; visual sphere radius=0.05
- added link wheel_link_br, mass 0.4; collision cylinder length=0.05 radius=0.05; visual sphere radius=0.05
- added link wheel_link_fl, mass 0.4; collision cylinder length=0.05 radius=0.05; visual sphere radius=0.05
- added link wheel_link_fr, mass 0.4; collision cylinder length=0.05 radius=0.05; visual sphere radius=0.05
- link base_link: mass 10.0 -> 22.0; geometry collision mesh filename=package://youbot_description/meshes/youbot_base/base_convex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; visual mesh filename=package://youbot_description/meshes/youbot_base/base.dae
Joints:
- added joint ar_marker_fixed_joint: type fixed, parent plate_link, child ar_marker_fixed, origin xyz=0.025 0 0 rpy=0 0 0
- added joint base_footprint_joint: type fixed, parent base_footprint, child base_link, origin xyz=0 0 0 rpy=0 0 0
- added joint base_laser_front_hokuyo_urg04_laser_joint: type fixed, parent base_link, child base_laser_front_link, origin xyz=0.3 0 -0.03 rpy=3.14 0 0, axis 0 1 0
- added joint caster_joint_bl: type continuous, parent base_link, child caster_link_bl, origin xyz=-0.228 0.158 -0.034 rpy=0 0 0, axis 0 0 1, limit effort=30 velocity=10
- added joint caster_joint_br: type continuous, parent base_link, child caster_link_br, origin xyz=-0.228 -0.158 -0.034 rpy=0 0 0, axis 0 0 1, limit effort=30 velocity=10
- added joint caster_joint_fl: type continuous, parent base_link, child caster_link_fl, origin xyz=0.228 0.158 -0.034 rpy=0 0 0, axis 0 0 1, limit effort=30 velocity=10
- added joint caster_joint_fr: type continuous, parent base_link, child caster_link_fr, origin xyz=0.228 -0.158 -0.034 rpy=0 0 0, axis 0 0 1, limit effort=30 velocity=10
- added joint plate_joint: type fixed, parent base_link, child plate_link, origin xyz=-0.159 0 0.046 rpy=0 0 0
- added joint wheel_joint_bl: type continuous, parent caster_link_bl, child wheel_link_bl, origin xyz=0.0 0.0 0.0 rpy=0 0 0, axis 0 1 0, limit effort=10 velocity=10
- added joint wheel_joint_br: type continuous, parent caster_link_br, child wheel_link_br, origin xyz=0.0 0.0 0.0 rpy=0 0 0, axis 0 1 0, limit effort=30 velocity=10
- added joint wheel_joint_fl: type continuous, parent caster_link_fl, child wheel_link_fl, origin xyz=0.0 0.0 0.0 rpy=0 0 0, axis 0 1 0, limit effort=30 velocity=10
- added joint wheel_joint_fr: type continuous, parent caster_link_fr, child wheel_link_fr, origin xyz=0.0 0.0 0.0 rpy=0 0 0, axis 0 1 0, limit effort=30 velocity=10
- joint arm_joint_0: origin xyz=0 0 0 rpy=0 0 0 -> xyz=0.143 0 0.046 rpy=0 0 0
- joint arm_joint_1: origin xyz=0.024 0 0.096 rpy=0 0 2.96705972839 -> xyz=0.024 0 0.115 rpy=0 0 -2.96705972839
- joint arm_joint_2: axis 0 1 0 -> 0 0 1; origin xyz=0.033 0 0.019 rpy=0 -1.1344640138 0 -> xyz=0.033 0 0 rpy=-1.57079632679 0 1.57079632679

File: urdf/youbot_arm/arm.urdf.xacro (robot description, xacro)
@@ -45,5 +45,5 @@
 			<parent link="${name}_link_0"/>
 			<child link="${name}_link_1"/>
-      <axis xyz="0 0 1"/>
+      <axis xyz="0 0 -1"/>
 			<!--<calibration rising="${arm_1_ref}" falling="${arm_1_ref}"/>-->
 			<dynamics damping="1" friction="1" />
@@ -68,5 +68,5 @@
 					<mesh filename="package://youbot_description/meshes/youbot_arm/arm1.dae" />
 				</geometry>
-				<material name="Orange" />
+				<!--<material name="Orange" />-->
 			</visual>
 			<collision>
