Commit message: moved origin of the plate down to better match the real robot

File: robots/youbot.urdf.xacro (robot description, xacro)
@@ -31,5 +31,5 @@
   <xacro:youbot_base name="base"/>
   <xacro:youbot_plate name="plate" parent="base_link">
-    <origin xyz="-0.159 0 0.046" rpy="0 0 0" />
+    <origin xyz="-0.159 0 0.021" rpy="0 0 0" />
   </xacro:youbot_plate>
   <xacro:youbot_arm name="arm" parent="base_link">

Commit message: Cleaned up package of temporary and outdated files.  Also modified controllers and controller_manager.  Extensive work to URDFs to incorporate stock downloaded parts from youbot-store.

File: robots/youbot.urdf.xacro (robot description, xacro)
@@ -37,5 +37,5 @@
   </xacro:youbot_arm>
   <xacro:youbot_gripper name="gripper" parent="arm_link_5">
-    <origin xyz="0 0 0" rpy="0 0 0" />
+    <origin xyz="-0.0027 0 .016" rpy="0 ${-M_PI/2} ${M_PI}" />
   </xacro:youbot_gripper>
 </robot>

File: urdf/youbot_arm/arm.urdf.xacro (robot description, xacro)
@@ -42,5 +42,5 @@
 		<!-- joint between arm_0_link and arm_1_link -->
 		<joint name="${name}_joint_1" type="revolute">
-			<origin xyz="0.024 0 0.096" rpy="0 0 ${170 * M_PI / 180}"/>
+			<origin xyz="0.024 0 0.115" rpy="0 0 ${170 * M_PI / 180}"/>
 			<parent link="${name}_link_0"/>
 			<child link="${name}_link_1"/>
@@ -64,7 +64,7 @@
 			</inertial>
 			<visual>
-				<origin xyz="0 0 0" rpy="0 0 0" />
-				<geometry>
-					<mesh filename="package://youbot_description/meshes/youbot_arm/arm1.dae" />
+				<origin xyz="0 0 0" rpy="${M_PI} 0 0" />
+				<geometry>
+				  <mesh filename="package://youbot_description/meshes/youbot_arm/arm1.dae" />
 				</geometry>
 				<!--<material name="Orange" />-->
@@ -72,7 +72,7 @@
 			<collision>
 				<!--<origin xyz="0 0 -0.003" rpy="0 0 0" />-->
-				<origin xyz="0 0 0" rpy="0 0 0" />
-				<geometry>
-					<mesh filename="package://youbot_description/meshes/youbot_arm/arm1_convex.dae" />
+				<origin xyz="0 0 0" rpy="${M_PI} 0 0" />
+				<geometry>
+					<mesh filename="package://youbot_description/meshes/youbot_arm/arm_joint_1_convex.stl" />
 					<!--<cylinder length="0.102" radius="0.080"/>-->
 				</geometry>
@@ -84,5 +84,5 @@
 		<!-- joint between arm_1_link and arm_2_link -->
 		<joint name="${name}_joint_2" type="revolute">
-			<origin xyz="0.033 0 0.019" rpy="0 ${-65 * M_PI / 180} 0"/>
+			<origin xyz="0.033 0 0" rpy="0 ${-65 * M_PI / 180} 0"/>
 			<parent link="${name}_link_1"/>
 			<child link="${name}_link_2"/>
@@ -99,7 +99,7 @@
 			</inertial>
 			<visual>
-			<origin xyz="0 -0.032 0.078" rpy="0 0 0" />
-				<geometry>
-					<mesh filename="package://youbot_description/meshes/youbot_arm/arm2.dae" />
+			<origin xyz="0 0 0" rpy="${- M_PI / 2} ${- M_PI / 2} 0" />
+				<geometry>
+				  <mesh filename="package://youbot_description/meshes/youbot_arm/arm2.dae" />
 				</geometry>
 				<material name="Orange" />
@@ -107,7 +107,7 @@
 			<collision>
 				<!--<origin xyz="0.001 -0.041 0.074" rpy="0 0 0" />-->
-				<origin xyz="0 -0.032 0.078" rpy="0 0 0" />
-				<geometry>
-					<mesh filename="package://youbot_description/meshes/youbot_arm/arm2_convex.dae" />
+				<origin xyz="0 0 0" rpy="${- M_PI / 2} ${- M_PI / 2} 0" />
+				<geometry>
+					<mesh filename="package://youbot_description/meshes/youbot_arm/arm_joint_2_convex.stl" />
 					<!--<box size="0.074 0.082 0.222"/>-->
 				</geometry>
@@ -142,7 +142,7 @@
 			</inertial>
 			<visual>
-				<origin xyz="0.000 0.028 0.079" rpy="0 0 0" />
-				<geometry>
-					<mesh filename="package://youbot_description/meshes/youbot_arm/arm3.dae" />
+				<origin xyz="0 0 0" rpy="${M_PI / 2} 0 ${M_PI}" />
+				<geometry>
+				  <mesh filename="package://youbot_description/meshes/youbot_arm/arm3.dae" />
 				</geometry>
 				<material name="Orange" />
@@ -150,7 +150,7 @@
 			<collision>
 				<!--<origin xyz="0.000 0.025 0.067" rpy="0 0 0" />-->
-				<origin xyz="0.000 0.028 0.079" rpy="0 0 0" />
-				<geometry>
-					<mesh filename="package://youbot_description/meshes/youbot_arm/arm3_convex.dae" />
+				<origin xyz="0 0 0" rpy="${M_PI / 2} 0 ${M_PI}" />
+				<geometry>
+					<mesh filename="package://youbot_description/meshes/youbot_arm/arm_joint_3_convex.stl" />
 					<!--<box size="0.064 0.054 0.192"/>-->
 				</geometry>
@@ -177,7 +177,7 @@
 			</inertial>
 			<visual>
-				<origin xyz="0 -0.010 0.029" rpy="0 0 0"/>
-				<geometry>
-					<mesh filename="package://youbot_description/meshes/youbot_arm/arm4.dae" />
+				<origin xyz="0 0 0" rpy="${M_PI / 2} 0 ${M_PI}"/>
+				<geometry>
+				  <mesh filename="package://youbot_description/meshes/youbot_arm/arm4.dae" />
 				</geometry>
 				<material name="Orange" />
@@ -185,7 +185,7 @@
 			<collision>
 				<!--<origin xyz="0 0 0.026" rpy="0 0 0" />-->
-				<origin xyz="0 -0.010 0.029" rpy="0 0 0"/>
-				<geometry>
-					<mesh filename="package://youbot_description/meshes/youbot_arm/arm4_convex.dae" />
+				<origin xyz="0 0 0" rpy="${M_PI / 2} 0 ${M_PI}"/>
+				<geometry>
+					<mesh filename="package://youbot_description/meshes/youbot_arm/arm_joint_4_convex.stl" />
 					<!--<box size="0.058 0.100 0.118"/>-->
 				</geometry>
@@ -197,5 +197,5 @@
 		<!-- joint between arm_4_link and arm_5_link -->
 		<joint name="${name}_joint_5" type="revolute">
-			<origin xyz="-0.002 0 0.130" rpy="0 0 ${167.5 * M_PI / 180}" />
+			<origin xyz="0 0 0.114" rpy="0 0 ${167.5 * M_PI / 180}" />
 			<parent link="${name}_link_4"/>
 			<child link="${name}_link_5"/>
@@ -212,14 +212,14 @@
 			</inertial>
 			<visual>
-				<origin xyz="0.003 0 -0.034" rpy="0 0 0" />
-				<geometry>
-					<mesh filename="package://youbot_description/meshes/youbot_arm/arm5.dae" />
+				<origin xyz="0 0 0" rpy="0 0 0" />
+				<geometry>
+				  <mesh filename="package://youbot_description/meshes/youbot_arm/arm5.dae" />
 				</geometry>
 				<material name="DarkGrey" />
 			</visual>
 			<collision>
-				<origin xyz="0.003 0 -0.034" rpy="0 0 0" />
-				<geometry>
-					<mesh filename="package://youbot_description/meshes/youbot_arm/arm5_convex.dae" />
+				<origin xyz="0 0 0" rpy="0 0 0" />
+				<geometry>
+					<mesh filename="package://youbot_description/meshes/youbot_arm/arm_joint_5_convex.stl" />
 					<!--<box size="0.054 0.096 0.030"/>-->
 				</geometry>

File: urdf/youbot_base/base.urdf.xacro (robot description, xacro)
@@ -122,8 +122,7 @@
       			<visual>
         			<origin xyz="0 0 0" rpy="0 0 0" />
-					<!--<mesh filename="package://youbot_description/meshes/youbot_base/youbot_wheel.stl" />-->
-				<geometry>
-					<sphere radius="${wheel_radius}"/>
-				</geometry>
+				      <geometry>
+					      <mesh filename="package://youbot_description/meshes/youbot_base/front-left_wheel.dae" />
+				      </geometry>
        				<material name="Orange" />
       			</visual>
@@ -171,8 +170,7 @@
       			<visual>
         			<origin xyz="0 0 0" rpy="0 0 0" />
-				<geometry>
-          				<!--<mesh filename="package://youbot_description/meshes/youbot_base/youbot_wheel.stl" />-->
-					<sphere radius="${wheel_radius}"/>
-        			</geometry>
+				      <geometry>
+					      <mesh filename="package://youbot_description/meshes/youbot_base/front-right_wheel.dae" />
+				      </geometry>
        				<material name="Orange" />
       			</visual>
@@ -221,8 +219,7 @@
       			<visual>
         			<origin xyz="0 0 0" rpy="0 0 0" />
-				<geometry>
-          				<!--<mesh filename="package://youbot_description/meshes/youbot_base/youbot_wheel.stl" />-->
-					<sphere radius="${wheel_radius}"/>
-        			</geometry>
+				      <geometry>
+					      <mesh filename="package://youbot_description/meshes/youbot_base/back-left_wheel.dae" />
+				      </geometry>
        				<material name="Orange" />
       			</visual>
@@ -273,8 +270,7 @@
       			<visual>
         			<origin xyz="0 0 0" rpy="0 0 0" />
-				<geometry>
-          				<!--<mesh filename="package://youbot_description/meshes/youbot_base/youbot_wheel.stl" />-->
-					<sphere radius="${wheel_radius}"/>
-        			</geometry>
+				      <geometry>
+					      <mesh filename="package://youbot_description/meshes/youbot_base/back-right_wheel.dae" />
+				      </geometry>
        				<material name="Orange" />
       			</visual>

File: urdf/youbot_gripper/gripper.urdf.xacro (robot description, xacro)
@@ -9,7 +9,7 @@
 <!--	<include filename="$(find youbot_description)/urdf/sensors/asus_xtion_camera.urdf.xacro" /> -->
 	<xacro:macro name="youbot_gripper" params="parent name *origin">
-		<!-- joint between arm_7_link and sdh_palm_link -->
+		<!-- joint between arm_link_5 and sdh_palm_link -->
 		<joint name="${name}_palm_joint" type="fixed" >
-			<insert_block name="origin" />
+      <insert_block name="origin" />
 			<parent link="${parent}" />
 			<child link="${name}_palm_link" />
@@ -17,17 +17,17 @@
 		<link name="${name}_palm_link">
 			<inertial>
-				<origin xyz="0 0 0" rpy="0 0 0"/>
+				<origin xyz="0 0 0" rpy="${M_PI} ${-M_PI / 2}  0"/>
 				<mass value="0.1"/>
 				<inertia ixx="0.01" ixy="0" ixz="0" iyy="0.01" iyz="0" izz="0.01" />
 			</inertial>
 			<visual>
-				<origin xyz="0 0 0" rpy="0 0 0" />
+				<origin xyz="0 0 0" rpy="${M_PI} ${-M_PI / 2} 0" />
 				<geometry>
 					<mesh filename="package://youbot_description/meshes/youbot_gripper/palm.dae" />
 				</geometry>
-				<material name="youbot/Black" />
+				<material name="Black" />
 			</visual>
 			<collision>
-				<origin xyz="0 0 0" rpy="0 0 0" />
+				<origin xyz="0 0 0" rpy="${M_PI} ${-M_PI / 2} 0" />
 				<geometry>
 					<!--<box size="0.050 0.094 0.054"/>-->
@@ -50,5 +50,5 @@
 -->
 			<collision>
-				<origin xyz="0 0 0" rpy="0 0 0"/>
+				<origin xyz="0 0 0" rpy="0 ${-M_PI / 2} 0"/>
 				<geometry>
 					<box size="0.07 0.2 0.06"/>
@@ -57,11 +57,11 @@
 		</link>
 		<joint name="${name}_camera_collision_box_joint" type="fixed">
-			<origin xyz="0.05 0 0.02" rpy="0 ${M_PI/2} 0"/>
+			<origin xyz="0 0 0.060" rpy="0 0 0"/>
 			<parent link="${name}_palm_link"/>
 			<child link ="${name}_camera_collision_box_link"/>
-			<axis xyz="0 -1 0"/>
+			<axis xyz="0 1 0"/>
 		</joint>
 		<joint name="${name}_finger_joint_l" type="prismatic">
-			<origin xyz="0.004 0.008 0.046" rpy="0 0 ${M_PI}" />
+			<origin xyz="0.046 0.010 0.003 " rpy="0 ${-M_PI / 2} ${M_PI}" />
 			<parent link="${name}_palm_link"/>
 			<child link="${name}_finger_link_l"/>
@@ -82,5 +82,5 @@
 					<mesh filename="package://youbot_description/meshes/youbot_gripper/finger.dae" />
 				</geometry>
-				<material name="youbot/Black" />
+				<material name="Black" />
 			</visual>
 			<collision>
@@ -95,6 +95,6 @@
 			<material>Black</material>
 		</gazebo>
-               <joint name="${name}_finger_joint_r" type="prismatic">
-			<origin xyz="0.004 -0.008 0.046" rpy="0 0 0" />
+    <joint name="${name}_finger_joint_r" type="prismatic">
+			<origin xyz="0.046 -0.010 0.003" rpy="0 ${M_PI / 2} 0" />
 			<parent link="${name}_palm_link"/>
 			<child link="${name}_finger_link_r"/>
@@ -115,5 +115,5 @@
 					<mesh filename="package://youbot_description/meshes/youbot_gripper/finger.dae" />
 				</geometry>
-				<material name="youbot/Black" />
+				<material name="Black" />
 			</visual>
 			<collision>

Commit message: corrected the plate location

File: robots/youbot.urdf.xacro (robot description, xacro)
@@ -31,5 +31,5 @@
   <xacro:youbot_base name="base"/>
   <xacro:youbot_plate name="plate" parent="base_link">
-    <origin xyz="-0.159 0 0.03" rpy="0 0 0" />
+    <origin xyz="-0.159 0 0.055" rpy="0 0 0" />
   </xacro:youbot_plate>
   <xacro:youbot_arm name="arm" parent="base_link">

File: urdf/youbot_plate/plate.urdf.xacro (robot description, xacro)
@@ -37,5 +37,5 @@
 		<!-- fixed ar marker attached to plate -->
                 <joint name="ar_marker_fixed_joint" type="fixed">
-			<origin xyz="0.025 0 0.025" rpy="0 0 0" />
+			<origin xyz="0.025 0 0" rpy="0 0 0" />
 			<parent link="${name}_link" />
 			<child link="ar_marker_fixed" />
