Commit message: Editted some URDFs

File: gazebo/gazebo.urdf.xacro (robot description, xacro)
@@ -4,4 +4,5 @@
        xmlns:interface="http://playerstage.sourceforge.net/gazebo/xmlschema/#interface">
   <gazebo>
+  <!--
     <controller:gazebo_ros_controller_manager name="gazebo_ros_controller_manager" plugin="libgazebo_ros_controller_manager.so">
       <alwaysOn>true</alwaysOn>
@@ -22,4 +23,5 @@
       <chargeVoltage>16.41</chargeVoltage>
     </controller:gazebo_ros_power_monitor>
+  -->
   </gazebo>
 </robot>

File: urdf/sensors/hokuyo_urg04_laser.gazebo.xacro (robot description, xacro)
@@ -6,25 +6,21 @@
   <xacro:macro name="hokuyo_urg04_laser_gazebo" params="name ros_topic update_rate min_angle max_angle">
     <gazebo reference="${name}_link">
-      <sensor:ray name="${name}">
-        <rayCount>640</rayCount>
-        <rangeCount>640</rangeCount>
-        <laserCount>1</laserCount>
-        <origin>0.0 0.0 0.0</origin>
-        <displayRays>false</displayRays>
-        <minAngle>${min_angle*180.0/M_PI}</minAngle>
-        <maxAngle>${max_angle*180.0/M_PI}</maxAngle>
-        <minRange>0.05</minRange>
-        <maxRange>5.6</maxRange>
-        <resRange>0.36</resRange>
-        <updateRate>${update_rate}</updateRate>
-        <controller:gazebo_ros_laser name="gazebo_ros_${name}_controller" plugin="libgazebo_ros_laser.so">
-          <gaussianNoise>0.000</gaussianNoise>
-          <alwaysOn>true</alwaysOn>
-          <updateRate>${update_rate}</updateRate>
-          <topicName>${ros_topic}</topicName>
-          <frameName>/${name}_link</frameName>
-          <interface:laser name="gazebo_ros_${name}_iface" />
-        </controller:gazebo_ros_laser>
-      </sensor:ray>
+      <sensor name="${name}" type="ray">
+	<ray>
+	  <scan>
+	    <horizontal>
+		<samples>640</samples>
+		<resolution>1.0</resolution>
+		<min_angle>${min_angle*180.0/M_PI}</min_angle>
+		<max_angle>${max_angle*180.0/M_PI}</max_angle>
+	    </horizontal>
+	  </scan>
+	  <range>
+		<min>0.05</min>
+		<max>5.6</max>
+		<resolution>0.36</resolution>
+	  </range>
+	</ray>
+      </sensor>
     </gazebo>
   </xacro:macro>

File: urdf/youbot_arm/arm.gazebo.xacro (robot description, xacro)
@@ -7,25 +7,25 @@
 		<gazebo reference="${name}_link_0">
 			<material value="youbot/DarkGrey" />
-			<turnGravityOff>false</turnGravityOff>
+			<gravity>false</gravity>
 		</gazebo>
 		<gazebo reference="${name}_link_1">
 			<!--<material value="youbot/Orange" />-->
-			<turnGravityOff>false</turnGravityOff>
+			<gravity>false</gravity>
 		</gazebo>
 		<gazebo reference="${name}_link_2">
 			<!--<material value="youbot/Orange" />-->
-			<turnGravityOff>false</turnGravityOff>
+			<gravity>false</gravity>
 		</gazebo>
 		<gazebo reference="${name}_link_3">
 			<!--<material value="youbot/Orange" />-->
-			<turnGravityOff>false</turnGravityOff>
+			<gravity>false</gravity>
 		</gazebo>
 		<gazebo reference="${name}_link_4">
 			<!--<material value="youbot/Orange" />-->
-			<turnGravityOff>false</turnGravityOff>
+			<gravity>false</gravity>
 		</gazebo>
 		<gazebo reference="${name}_link_5">
 			<!--<material value="youbot/DarkGrey" />-->
-			<turnGravityOff>false</turnGravityOff>
+			<gravity>false</gravity>
 		</gazebo>
 	</xacro:macro>

File: urdf/youbot_gripper/gripper.gazebo.xacro (robot description, xacro)
@@ -7,15 +7,15 @@
 		<gazebo reference="${name}_palm_link">
 			<material>Gazebo/Black</material>
-			<turnGravityOff>false</turnGravityOff>
+			<gravity>false</gravity>
 			<selfCollide>true</selfCollide>
 		</gazebo>
 		<gazebo reference="${name}_finger_l_link">
 			<material>Gazebo/Black</material>
-			<turnGravityOff>false</turnGravityOff>
+			<gravity>false</gravity>
 			<selfCollide>true</selfCollide>
 		</gazebo>
 		<gazebo reference="${name}_finger_r_link">
 			<material>Gazebo/Black</material>
-			<turnGravityOff>false</turnGravityOff>
+			<gravity>false</gravity>
 			<selfCollide>true</selfCollide>
 		</gazebo>
