Commit message: Modified youbot_controllers with new pluginlib declaration (export)

File: urdf/sensors/asus_xtion_camera.gazebo.xacro (robot description, xacro)
@@ -10,13 +10,20 @@
 <xacro:macro name="asus_xtion_depth_camera_gazebo" params="name">
   <gazebo reference="${name}_depth_frame">
-    <sensor:camera name="${name}_depth_frame_sensor">
-      <imageFormat>R8G8B8</imageFormat>
-      <imageSize>640 480</imageSize>
-      <hfov>57</hfov>
-      <nearClip>0.01</nearClip>
-      <farClip>5</farClip>
-      <updateRate>20.0</updateRate>
-      <baseline>0.2</baseline>
-      <controller:gazebo_ros_camera name="${name}_depth_frame_controller" plugin="libgazebo_ros_camera.so">
+    <sensor type="camera" name="${name}_depth_frame_sensor">
+      <camera>
+	<horizontal_fov>57.0</horizontal_fov>
+	<image>
+	  <format>R8G8B8</format>
+          <width>640</width>
+	  <height>480</height>
+	</image>
+        <clip>
+	  <near>0.01</near>
+	  <far>5</far>
+	</clip>
+      </camera>
+      <update_rate>20.0</update_rate>
+      <!--<baseline>0.2</baseline>-->
+      <plugin name="${name}_depth_frame_controller" filename="libgazebo_ros_camera.so">
         <alwaysOn>true</alwaysOn>
         <updateRate>20.0</updateRate>
@@ -33,19 +40,26 @@
         <distortion_t1>0.00000001</distortion_t1>
         <distortion_t2>0.00000001</distortion_t2>
-      </controller:gazebo_ros_camera>
-    </sensor:camera>
+      </plugin>
+    </sensor>
   </gazebo>
 </xacro:macro>
 <xacro:macro name="asus_xtion_rgb_camera_gazebo" params="name">
   <gazebo reference="${name}_rgb_frame">
-    <sensor:camera name="${name}_rgb_frame_sensor">
-      <imageFormat>R8G8B8</imageFormat>
-      <imageSize>640 480</imageSize>
-      <hfov>57</hfov>
-      <nearClip>0.01</nearClip>
-      <farClip>5</farClip>
-      <updateRate>20.0</updateRate>
-      <baseline>0.2</baseline>
-      <controller:gazebo_ros_camera name="${name}_rgb_frame_controller" plugin="libgazebo_ros_camera.so">
+    <sensor type="camera" name="${name}_rgb_frame_sensor">
+      <camera>
+	<image>
+	  <format>R8G8B8</format>
+          <width>640</width>
+	  <height>480</height>
+	</image>
+        <horizontal_fov>57</horizontal_fov>
+        <clip>
+	  <near>0.01</near>
+	  <far>5</far>
+	</clip>
+      </camera>
+      <update_rate>20.0</update_rate>
+      <!--<baseline>0.2</baseline>-->
+      <plugin name="${name}_rgb_frame_controller" filename="libgazebo_ros_camera.so">
         <alwaysOn>true</alwaysOn>
         <updateRate>20.0</updateRate>
@@ -59,6 +73,6 @@
         <distortion_t1>0.00000001</distortion_t1>
         <distortion_t2>0.00000001</distortion_t2>
-      </controller:gazebo_ros_camera>
-    </sensor:camera>
+      </plugin>
+    </sensor>
   </gazebo>
 </xacro:macro>

File: urdf/sensors/hokuyo_urg04_laser.gazebo.xacro (robot description, xacro)
@@ -22,4 +22,12 @@
 	  </range>
 	</ray>
+	<plugin name="gazebo_ros_${name}_controller" filename="libgazebo_ros_laser.so">
+	  <gaussianNoise>0.000</gaussianNoise>
+	  <alwaysOn>true</alwaysOn>
+	  <updateRate>${update_rate}</updateRate>
+	  <topicName>${ros_topic}</topicName>
+	  <frameName>/${name}_link</frameName>
+	  <interface:laser name="gazebo_ros_${name}_iface" />
+        </plugin>
       </sensor>
     </gazebo>

File: urdf/youbot_arm/arm.gazebo.xacro (robot description, xacro)
@@ -5,26 +5,22 @@
        xmlns:xacro="http://ros.org/wiki/xacro">
 	<xacro:macro name="youbot_arm_gazebo" params="name">
-		<gazebo reference="${name}_link_0">
-			<material value="youbot/DarkGrey" />
+		<gazebo>
+		  <link name="${name}_link_0">
 			<gravity>false</gravity>
+		  </link>
 		</gazebo>
 		<gazebo reference="${name}_link_1">
-			<!--<material value="youbot/Orange" />-->
 			<gravity>false</gravity>
 		</gazebo>
 		<gazebo reference="${name}_link_2">
-			<!--<material value="youbot/Orange" />-->
 			<gravity>false</gravity>
 		</gazebo>
 		<gazebo reference="${name}_link_3">
-			<!--<material value="youbot/Orange" />-->
 			<gravity>false</gravity>
 		</gazebo>
 		<gazebo reference="${name}_link_4">
-			<!--<material value="youbot/Orange" />-->
 			<gravity>false</gravity>
 		</gazebo>
 		<gazebo reference="${name}_link_5">
-			<!--<material value="youbot/DarkGrey" />-->
 			<gravity>false</gravity>
 		</gazebo>

File: urdf/youbot_base/base.gazebo.xacro (robot description, xacro)
@@ -38,5 +38,5 @@
 	<!-- position controller -->
 		<gazebo>
-      			<controller:gazebo_ros_p3d name="p3d_base_controller" plugin="libgazebo_ros_p3d.so">
+      			<plugin name="p3d_base_controller" filename="libgazebo_ros_p3d.so">
         			<alwaysOn>true</alwaysOn>
         			<updateRate>100.0</updateRate>
@@ -48,5 +48,5 @@
         			<rpyOffsets>0 0 0</rpyOffsets>
         			<interface:position name="p3d_base_position"/>
-      			</controller:gazebo_ros_p3d>
+      			</plugin>
       			<canonicalBody>base_footprint</canonicalBody>
     		</gazebo>

File: urdf/youbot_gripper/gripper.urdf.xacro (robot description, xacro)
@@ -26,5 +26,5 @@
 					<mesh filename="package://youbot_description/meshes/youbot_gripper/palm.dae" />
 				</geometry>
-				<material name="Black" />
+				<material name="youbot/Black" />
 			</visual>
 			<collision>
@@ -59,5 +59,5 @@
 					<mesh filename="package://youbot_description/meshes/youbot_gripper/finger.dae" />
 				</geometry>
-				<material name="Black" />
+				<material name="youbot/Black" />
 			</visual>
 			<collision>
@@ -92,5 +92,5 @@
 					<mesh filename="package://youbot_description/meshes/youbot_gripper/finger.dae" />
 				</geometry>
-				<material name="Black" />
+				<material name="youbot/Black" />
 			</visual>
 			<collision>
