Commit message: removed base from camera, set its parent to xtion_pose, added fixed AR tag to plate

File: urdf/sensors/asus_xtion_camera.urdf.xacro (robot description, xacro)
@@ -19,4 +19,5 @@
   </xacro:macro>
   <xacro:macro name="asus_xtion_camera" params="name parent *origin tilt">
+<!--
   	<link name="${name}_foot_link">
       <inertial>
@@ -68,8 +69,9 @@
      	<parent link="${name}_foot_link"/>
      	<child link="${name}_tilt_link"/>
-   	<!--<axis xyz="0 1 0"/>-->
-    	<origin xyz="0 0 0.0075" rpy="0 ${tilt} 0"/>
-	<!--<limit effort="100" lower="-0.541052068" upper="0.541052068" velocity="1.0"/>-->
-    </joint>
+--> 	<!--<axis xyz="0 1 0"/>-->
+<!--    	<origin xyz="0 0 0.0075" rpy="0 ${tilt} 0"/>
+-->	<!--<limit effort="100" lower="-0.541052068" upper="0.541052068" velocity="1.0"/>-->
+<!--    </joint>
+-->
     <link name="${name}_camera">
       <inertial>
@@ -94,5 +96,6 @@
     <joint name="${name}_camera_joint" type="fixed">
       <origin xyz="0 0.03 0.03" rpy="0 0 0" />
-      <parent link="${name}_tilt_link"/>
+      <parent link = "${parent}"/>
+<!--      <parent link= "${name}_tilt_link"/> -->
       <child link="${name}_camera"/>
     </joint>

File: urdf/youbot_gripper/gripper.urdf.xacro (robot description, xacro)
@@ -105,7 +105,7 @@
 			<material>Black</material>
 		</gazebo>
-		<!-- asus xtion camera -->
-		<xacro:asus_xtion_camera name="openni" parent="gripper_palm_link" tilt="0.0">
-		  <origin xyc="0.01 0.0 0.0" rpy="0 ${M_PI/2} 0.0" />
+                <!-- asus xtion camera -->
+		<xacro:asus_xtion_camera name="xtion" parent="xtion_pose" tilt="0.0">
+		  <origin xyc="0.00 0.0 0.0" rpy="0 0 0" />
                 </xacro:asus_xtion_camera>
 		<!-- extensions -->

File: urdf/youbot_plate/plate.urdf.xacro (robot description, xacro)
@@ -35,4 +35,24 @@
 		</gazebo>
 		<!-- extensions -->
+		<!-- fixed ar marker attached to plate -->
+                <joint name="ar_marker_fixed_joint" type="fixed">
+			<origin xyz="0 0 0.025" rpy="0 0 0" />
+			<parent link="${name}_link" />
+			<child link="ar_marker_fixed" />
+		</joint>
+		<link name="ar_marker_fixed">
+			<visual>
+				<origin xyz="0 0 0" rpy="0 0 0" />
+				<geometry>
+					<box size="0.08 0.08 0.003" />
+				</geometry>
+			</visual>
+			<collision>
+				<origin xyz="0 0 0" rpy="0 0 0" />
+				<geometry>
+					<box size="0.08 0.08 0.003" />
+				</geometry>
+			</collision>
+		</link>
 	</xacro:macro>
 </robot>

Commit message: Reacquired missing asus_xtion_camera.urdf.xacro file

File: urdf/sensors/asus_xtion_camera.urdf.xacro (robot description, xacro)
@@ -1,4 +1,9 @@
 <?xml version="1.0"?>
-<root xmlns:xacro="http://playerstage.sourceforge.net/gazebo/xmlschema/#interface">
+<robot xmlns:sensor="http://playerstage.sourceforge.net/gazebo/xmlschema/#sensor"
+       xmlns:controller="http://playerstage.sourceforge.net/gazebo/xmlschema/#controller"
+       xmlns:interface="http://playerstage.sourceforge.net/gazebo/xmlschema/#interface"
+       xmlns:xacro="http://playerstage.sourceforge.net/gazebo/xmlschema/#interface"
+       name="xtion" >
+  <property name="M_PI" value="3.14159"/>.
   <include filename="$(find youbot_description)/urdf/sensors/asus_xtion_camera.gazebo.xacro" />
   <property name="eye_x_offset" value="0.03" />
@@ -18,58 +23,5 @@
 	</joint>
   </xacro:macro>
-  <xacro:macro name="asus_xtion_camera" params="name parent *origin tilt">
-  	<link name="${name}_foot_link">
-      <inertial>
-        <mass value="0.05" />
-        <origin xyz="0 0 0" rpy="0 0 0"/>
-        <inertia ixx="0.0001" ixy="0" ixz="0" iyy="0.0001" iyz="0" izz="0.0001" />
-      </inertial>
-      <visual>
-        <origin xyz="0.01 0 0" rpy="${M_PI/2} 0 ${M_PI/2}" />
-        <geometry>
-           <mesh filename="package://youbot_description/meshes/sensors/asus_xtion_pro_live_base.dae" scale="0.0004 0.0007 0.001"/>
-        </geometry>
-        <material name="Black" />
-      </visual>
-      <collision>
-        <origin xyz="0.01 0 0" rpy="${M_PI/2} 0 ${M_PI/2}" />
-        <geometry>
-           <mesh filename="package://youbot_description/meshes/sensors/asus_xtion_pro_live_base.dae" scale="0.0004 0.0007 0.001"/>
-        </geometry>
-      </collision >
-    </link>
-    <joint name="${name}_foot_joint" type="fixed">
-      <insert_block name="origin" />
-      <parent link="${parent}"/>
-      <child link="${name}_foot_link"/>
-    </joint>
-    <link name="${name}_tilt_link">
-      <inertial>
-        <mass value="0.01" />
-        <origin xyz="0 0 0" rpy="0 0 0"/>
-        <inertia ixx="0.0001" ixy="0" ixz="0" iyy="0.0001" iyz="0" izz="0.0001" />
-      </inertial>
-      <visual>
-        <origin xyz="0 0 0.0075" rpy="0 0 0" />
-        <geometry>
-          <cylinder length="0.025" radius="0.005" />
-        </geometry>
-        <material name="Black" />
-      </visual>
-      <collision>
-        <origin xyz="0 0 0.0075" rpy="0 0 0" />
-        <geometry>
-          <cylinder length="0.025" radius="0.005" />
-        </geometry>
-        <material name="Black" />
-      </collision >
-    </link>
-    <joint name="asus_xtion_tilt_joint" type="fixed">
-     	<parent link="${name}_foot_link"/>
-     	<child link="${name}_tilt_link"/>
-   	<!--<axis xyz="0 1 0"/>-->
-    	<origin xyz="0 0 0.0075" rpy="0 ${tilt} 0"/>
-	<!--<limit effort="100" lower="-0.541052068" upper="0.541052068" velocity="1.0"/>-->
-    </joint>
+  <xacro:macro name="asus_xtion_camera" params="name *origin tilt">
     <link name="${name}_camera">
       <inertial>
@@ -92,10 +44,5 @@
       </collision >
     </link>
-    <joint name="${name}_camera_joint" type="fixed">
-      <origin xyz="0 0.03 0.03" rpy="0 0 0" />
-      <parent link="${name}_tilt_link"/>
-      <child link="${name}_camera"/>
-    </joint>
-    <xacro:asus_xtion_eye suffix="depth" parent="${name}">
+	<xacro:asus_xtion_eye suffix="depth" parent="${name}">
 		<origin xyz="${eye_x_offset} ${eye_y_offset - 0.02} 0" rpy="0 0 0" />
 	</xacro:asus_xtion_eye>
@@ -118,3 +65,6 @@
    <xacro:asus_xtion_camera_gazebo name="${name}" />
   </xacro:macro>
-</root>
+  <xacro:asus_xtion_camera name="xtion" tilt="0.0">
+     <origin xyz="0 0 0" rpy="0 0 0" />
+  </xacro:asus_xtion_camera>
+</robot>

Commit message: re-attached camera to youbot's urdf

File: urdf/sensors/asus_xtion_camera.urdf.xacro (robot description, xacro)
@@ -1,8 +1,7 @@
 <?xml version="1.0"?>
 <robot xmlns:sensor="http://playerstage.sourceforge.net/gazebo/xmlschema/#sensor"
-       xmlns:controller="http://playerstage.sourceforge.net/gazebo/xmlschema/#controller"
-       xmlns:interface="http://playerstage.sourceforge.net/gazebo/xmlschema/#interface"
-       xmlns:xacro="http://playerstage.sourceforge.net/gazebo/xmlschema/#interface"
-       name="xtion" >
+        xmlns:controller="http://playerstage.sourceforge.net/gazebo/xmlschema/#controller"
+        xmlns:interface="http://playerstage.sourceforge.net/gazebo/xmlschema/#interface"
+        xmlns:xacro="http://ros.org/wiki/xacro">
   <property name="M_PI" value="3.14159"/>.
   <include filename="$(find youbot_description)/urdf/sensors/asus_xtion_camera.gazebo.xacro" />
@@ -23,5 +22,5 @@
 	</joint>
   </xacro:macro>
-  <xacro:macro name="asus_xtion_camera" params="name *origin tilt">
+  <xacro:macro name="asus_xtion_camera" params="name parent *origin tilt">
     <link name="${name}_camera">
       <inertial>
@@ -44,4 +43,9 @@
       </collision >
     </link>
+    <joint name="${parent}_${name}_joint" type="fixed">
+      <insert_block name="origin" />
+      <parent link="${parent}" />
+      <child link="${name}_camera" />
+    </joint>
 	<xacro:asus_xtion_eye suffix="depth" parent="${name}">
 		<origin xyz="${eye_x_offset} ${eye_y_offset - 0.02} 0" rpy="0 0 0" />
@@ -65,6 +69,7 @@
    <xacro:asus_xtion_camera_gazebo name="${name}" />
   </xacro:macro>
-  <xacro:asus_xtion_camera name="xtion" tilt="0.0">
+<!--  <xacro:asus_xtion_camera name="xtion" tilt="0.0">
      <origin xyz="0 0 0" rpy="0 0 0" />
   </xacro:asus_xtion_camera>
+-->
 </robot>

File: urdf/youbot_gripper/gripper.urdf.xacro (robot description, xacro)
@@ -7,5 +7,5 @@
 	<include filename="$(find youbot_description)/urdf/youbot_gripper/gripper.transmission.xacro" />
 	<include filename="$(find youbot_description)/urdf/youbot_gripper/limits.urdf.xacro" />
-<!--	<include filename="$(find youbot_description)/urdf/sensors/asus_xtion_camera.urdf.xacro" /> -->
+	<include filename="$(find youbot_description)/urdf/sensors/asus_xtion_camera.urdf.xacro" />
 	<xacro:macro name="youbot_gripper" params="parent name *origin">
 		<!-- joint between arm_link_5 and sdh_palm_link -->
@@ -129,5 +129,5 @@
 		</gazebo>
                 <!-- asus xtion camera -->
-		<xacro:asus_xtion_camera name="xtion" tilt="0.0">
+		<xacro:asus_xtion_camera name="xtion" parent="${name}_palm_link" tilt="0.0">
                   <!-- AR_CALIBRATOR_START -->
 		  <origin xyz="0.02 -0.03 0.06" rpy="0 0 3.14" />

Commit message: moved camera collision box from gripper to camera, changed camera calibrator start flag in gripper urdf

File: urdf/sensors/asus_xtion_camera.urdf.xacro (robot description, xacro)
@@ -39,5 +39,8 @@
         <origin xyz="0.02 -0.03 0" rpy="${M_PI/2} 0 ${M_PI/2}" />
         <geometry>
-           <mesh filename="package://youbot_description/meshes/sensors/asus_xtion_pro_live_camera.dae" scale="0.001 0.001 0.001"/>
+   	  <box size="0.2 0.06 0.07"/>
+<!--
+	  <mesh filename="package://youbot_description/meshes/sensors/asus_xtion_pro_live_camera.dae" scale="0.001 0.001 0.001"/>
+-->
         </geometry>
       </collision >

File: urdf/youbot_gripper/gripper.urdf.xacro (robot description, xacro)
@@ -39,14 +39,6 @@
 			<material>Black</material>
 		</gazebo>
+<!--
 		<link name="${name}_camera_collision_box_link">
-<!--
-			<visual>
-				<origin xyz="0 0 0" rpy="0 0 0"/>
-				<geometry>
-					<box size="0.07 0.2 0.07"/>
-				</geometry>
-				<material name="youbot/Black"/>
-			</visual>
--->
 			<collision>
 				<origin xyz="0 0 0" rpy="0 ${-M_PI / 2} 0"/>
@@ -56,4 +48,6 @@
 			</collision>
 		</link>
+-->
+<!--
 		<joint name="${name}_camera_collision_box_joint" type="fixed">
 			<origin xyz="0 0 0.060" rpy="0 0 0"/>
@@ -62,4 +56,5 @@
 			<axis xyz="0 1 0"/>
 		</joint>
+-->
 		<joint name="${name}_finger_joint_l" type="prismatic">
 			<origin xyz="0.046 0.010 0.003 " rpy="0 ${-M_PI / 2} ${M_PI}" />
@@ -130,7 +125,6 @@
                 <!-- asus xtion camera -->
 		<xacro:asus_xtion_camera name="xtion" parent="${name}_palm_link" tilt="0.0">
-                  <!-- AR_CALIBRATOR_START -->
-		  <origin xyz="0.02 -0.03 0.06" rpy="0 0 3.14" />
-                  <!-- AR_CALIBRATOR_END -->
+                  <!-- AR_CALIBRATOR:EDIT_HERE -->
+                  <origin xyz="0.0197188 -0.0341838 0.0459352" rpy="0.0201114 0.00763208 3.0937" />
                 </xacro:asus_xtion_camera>
 		<!-- extensions -->
