Commit message: moved plate and ar_marker_fixed to better match their positions on the actual robot

File: urdf/youbot_plate/plate.urdf.xacro (robot description, xacro)
@@ -13,10 +13,10 @@
 		<link name="${name}_link">
 			<inertial>
-				<origin xyz="0 0 0" rpy="0 0 0"/>
+				<origin xyz="0 0 -0.025" rpy="0 0 0"/>
 				<mass value="1"/>
 				<inertia ixx="0.01" ixy="0" ixz="0" iyy="0.01" iyz="0" izz="0.01" />
 			</inertial>
 			<visual>
-				<origin xyz="0 0 0" rpy="0 0 0" />
+				<origin xyz="0 0 -0.025" rpy="0 0 0" />
 				<geometry>
 					<mesh filename="package://youbot_description/meshes/youbot_plate/plate.dae" />
@@ -25,5 +25,5 @@
 			</visual>
 			<collision>
-				<origin xyz="0 0 0" rpy="0 0 0" />
+				<origin xyz="0 0 -0.025" rpy="0 0 0" />
 				<geometry>
 					<mesh filename="package://youbot_description/meshes/youbot_plate/plate_convex.dae" />
@@ -37,5 +37,5 @@
 		<!-- fixed ar marker attached to plate -->
                 <joint name="ar_marker_fixed_joint" type="fixed">
-			<origin xyz="0 0 0.025" rpy="0 0 0" />
+			<origin xyz="0.025 0 0" rpy="0 0 0" /> <!-- z:0.025 for top of rviz plate -->
 			<parent link="${name}_link" />
 			<child link="ar_marker_fixed" />
@@ -45,8 +45,8 @@
 				<origin xyz="0 0 0" rpy="0 0 0" />
 				<geometry>
-					<box size="0.08 0.08 0.003" />
+					<box size="0.11 0.11 0.003" />
 				</geometry>
 			</visual>
-			<collision>
+<!--			<collision>
 				<origin xyz="0 0 0" rpy="0 0 0" />
 				<geometry>
@@ -54,5 +54,5 @@
 				</geometry>
 			</collision>
-		</link>
+-->		</link>
 	</xacro:macro>
 </robot>
