Commit message: Tweaked PID and updated controlleres

File: urdf/youbot_arm/arm.urdf.xacro (robot description, xacro)
@@ -229,4 +229,19 @@
 			<material>DarkGrey</material>
 		</gazebo>
+<!--
+    <joint name="${name}_joint_6_dummy" type="revolute">
+      <origin xyz="0 0 0" rpy="0 0 0"/>
+      <parent link="${name}_link_5"/>
+      <child link="${name}_link_6_dummy"/>
+      <axis xyz="0 0 1"/>
+      <limit effort="1" velocity="${M_PI / 2.0}" lower="0" upper="${2 * M_PI}" />
+    </joint>
+		<link name="${name}_link_6_dummy">
+			<inertial>
+				<mass value="0.001"/>
+				<xacro:link_5_inertia_tensor />
+			</inertial>
+		</link>
+-->
 		<!-- extensions -->
 		<xacro:youbot_arm_gazebo name="${name}" />

File: urdf/youbot_gripper/gripper.urdf.xacro (robot description, xacro)
@@ -7,5 +7,5 @@
 	<include filename="$(find youbot_description)/urdf/youbot_gripper/gripper.transmission.xacro" />
 	<include filename="$(find youbot_description)/urdf/youbot_gripper/limits.urdf.xacro" />
-	<include filename="$(find youbot_description)/urdf/sensors/asus_xtion_camera.urdf.xacro" />
+<!--	<include filename="$(find youbot_description)/urdf/sensors/asus_xtion_camera.urdf.xacro" /> -->
 	<xacro:macro name="youbot_gripper" params="parent name *origin">
 		<!-- joint between arm_7_link and sdh_palm_link -->
@@ -39,4 +39,27 @@
 			<material>Black</material>
 		</gazebo>
+		<link name="${name}_camera_collision_box_link">
+<!--
+			<visual>
+				<origin xyz="0 0 0" rpy="0 0 0"/>
+				<geometry>
+					<box size="0.07 0.2 0.07"/>
+				</geometry>
+				<material name="youbot/Black"/>
+			</visual>
+-->
+			<collision>
+				<origin xyz="0 0 0" rpy="0 0 0"/>
+				<geometry>
+					<box size="0.07 0.2 0.07"/>
+				</geometry>
+			</collision>
+		</link>
+		<joint name="${name}_camera_collision_box_joint" type="fixed">
+			<origin xyz="0.05 0 0.02" rpy="0 ${M_PI/2} 0"/>
+			<parent link="${name}_palm_link"/>
+			<child link ="${name}_camera_collision_box_link"/>
+			<axis xyz="0 -1 0"/>
+		</joint>
 		<joint name="${name}_finger_joint_l" type="prismatic">
 			<origin xyz="0.004 0.008 0.046" rpy="0 0 ${M_PI}" />
@@ -46,5 +69,5 @@
 			<dynamics damping="1.0" friction="1.0" />
 			<limit effort="1" velocity="0.1" lower="0" upper="${finger_joint}"/>
-                        <safety_controller k_position="20" k_velocity="25" soft_lower_limit="${threshold}" soft_upper_limit="${finger_joint_soft}" />
+                        <safety_controller k_position="20" k_velocity="25" soft_lower_limit="${gripper_threshold}" soft_upper_limit="${finger_joint_soft}" />
 		</joint>
 		<link name="${name}_finger_link_l">
@@ -79,5 +102,5 @@
 			<dynamics damping="1.0" friction="1.0" />
 			<limit effort="1" velocity="0.1" lower="0" upper="${finger_joint}"/>
-                        <safety_controller k_position="20" k_velocity="25" soft_lower_limit="${threshold}" soft_upper_limit="${finger_joint_soft}" />
+                        <safety_controller k_position="20" k_velocity="25" soft_lower_limit="${gripper_threshold}" soft_upper_limit="${finger_joint_soft}" />
 		</joint>
 		<link name="${name}_finger_link_r">
@@ -105,8 +128,9 @@
 			<material>Black</material>
 		</gazebo>
-		<!-- asus xtion camera -->
-		<xacro:asus_xtion_camera name="openni" parent="gripper_palm_link" tilt="0.0">
-		  <origin xyc="0.01 0.0 0.0" rpy="0 ${M_PI/2} 0.0" />
+                <!-- asus xtion camera -->
+<!--		<xacro:asus_xtion_camera name="xtion" tilt="0.0">
+		  <origin xyc="0.00 0.0 0.0" rpy="0 0 0" />
                 </xacro:asus_xtion_camera>
+-->
 		<!-- extensions -->
 		<xacro:youbot_gripper_gazebo name="${name}" />

File: urdf/youbot_gripper/limits.urdf.xacro (robot description, xacro)
@@ -3,7 +3,7 @@
 	<!-- common properties -->
 	<property name="M_PI" value="3.1415926535897931" />
-        <property name="threshold" value="0.001" />
+        <property name="gripper_threshold" value="0.001" />
 	<!-- fingers limits, values are in meters -->
 	<property name="finger_joint" value="${0.023 / 2.0}" />
-	<property name="finger_joint_soft" value="${(0.023 - threshold) / 2.0}" />
+	<property name="finger_joint_soft" value="${(0.023 - gripper_threshold) / 2.0}" />
 </robot>

Commit message: Downloaded new wheel meshes

File: urdf/youbot_arm/arm.urdf.xacro (robot description, xacro)
@@ -45,5 +45,5 @@
 			<parent link="${name}_link_0"/>
 			<child link="${name}_link_1"/>
-			<axis xyz="0 0 -1"/>
+      <axis xyz="0 0 1"/>
 			<!--<calibration rising="${arm_1_ref}" falling="${arm_1_ref}"/>-->
 			<dynamics damping="1" friction="1" />
@@ -68,5 +68,5 @@
 					<mesh filename="package://youbot_description/meshes/youbot_arm/arm1.dae" />
 				</geometry>
-				<!--<material name="Orange" />-->
+				<material name="Orange" />
 			</visual>
 			<collision>

File: urdf/youbot_gripper/gripper.urdf.xacro (robot description, xacro)
@@ -52,5 +52,5 @@
 				<origin xyz="0 0 0" rpy="0 0 0"/>
 				<geometry>
-					<box size="0.07 0.2 0.07"/>
+					<box size="0.07 0.2 0.06"/>
 				</geometry>
 			</collision>

Commit message: merging

File: urdf/youbot_arm/arm.urdf.xacro (robot description, xacro)
@@ -45,5 +45,5 @@
 			<parent link="${name}_link_0"/>
 			<child link="${name}_link_1"/>
-      <axis xyz="0 0 1"/>
+			<axis xyz="0 0 -1"/>
 			<!--<calibration rising="${arm_1_ref}" falling="${arm_1_ref}"/>-->
 			<dynamics damping="1" friction="1" />
