Commit message: modified the gripper so its fingers are in the middle position

File: urdf/youbot_gripper/gripper.urdf.xacro (robot description, xacro)
@@ -63,5 +63,5 @@
 		</joint>
 		<joint name="${name}_finger_joint_l" type="prismatic">
-			<origin xyz="0.004 0.008 0.046" rpy="0 0 ${M_PI}" />
+			<origin xyz="0.004 0.018 0.046" rpy="0 0 ${M_PI}" />
 			<parent link="${name}_palm_link"/>
 			<child link="${name}_finger_link_l"/>
@@ -96,5 +96,5 @@
 		</gazebo>
                <joint name="${name}_finger_joint_r" type="prismatic">
-			<origin xyz="0.004 -0.008 0.046" rpy="0 0 0" />
+			<origin xyz="0.004 -0.018 0.046" rpy="0 0 0" />
 			<parent link="${name}_palm_link"/>
 			<child link="${name}_finger_link_r"/>

Commit message: put the camera back on the gripper and added flags in gripper.urdf.xacro for the calibrator to modify the camera's position

File: urdf/youbot_gripper/gripper.urdf.xacro (robot description, xacro)
@@ -129,8 +129,9 @@
 		</gazebo>
                 <!-- asus xtion camera -->
-<!--		<xacro:asus_xtion_camera name="xtion" tilt="0.0">
-		  <origin xyc="0.00 0.0 0.0" rpy="0 0 0" />
+		<xacro:asus_xtion_camera name="xtion" tilt="0.0">
+                  <!-- AR_CALIBRATOR_START -->
+		  <origin xyz="0.02 -0.03 0.06" rpy="0 0 3.14" />
+                  <!-- AR_CALIBRATOR_END -->
                 </xacro:asus_xtion_camera>
--->
 		<!-- extensions -->
 		<xacro:youbot_gripper_gazebo name="${name}" />
